File: driver_module/driver_module.kicad_pcb (KiCad board)
At the start: 4 copper layers, 68.8 x 36 mm, 118 parts, among them J1 Power Input, J19 Conn_01x03, J2 Power Input, J21 Power Input, J4 Conn_02x06_Odd_Even, J5 Conn_02x06_Odd_Even, J6 Conn_01x06, Q1 Q_PNP_BEC, Q2 Q_PNP_BEC, Q3 Q_PNP_BEC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

Commit message: Generate Gerbers for JLC for Motor Driver Board.
Parts:
- removed J1: Power Input, parts:AMASS_XT60PW-F_1x02_P7.20mm_Horizontal
- removed J2: Power Input, parts:AMASS_XT60PW-M_1x02_P7.20mm_Horizontal
- added REF**: ESD-Logo_6.6x6mm_SilkScreen, Symbol:ESD-Logo_6.6x6mm_SilkScreen, F.Cu at (162.8, 90.9)
- added REF**: EastMakesLogo0.5x1CM, [Eastabrooka] Logos:EastMakesLogo0.5x1CM, F.Cu at (158.0, 87.3)
Other:
- board text removed: "Design by Sequoia Hope Alexander"
- board text removed: "Love"
- board text removed: "Many thanks to Daniel Theobald and our supporters on"
- board text removed: "Twisted Fields"
- board text removed: "everyone."
- board text removed: "github.com/ Twisted-Fields/rp2040-motor-controller"
- board text removed: "open collective for funding this work!"
