File: RP2040_base/RP2040_base.kicad_sch (KiCad schematic)
At the start: 321 parts, among them J1 CPU1 USB, J10 AUX GPIO 1, J11 CAN2 PLUG, J12 Conn_01x06, J13 ADC AUX 2, J14 AUX GPIO 2, J15 AUX Encoder, J16 Conn_02x05_Odd_Even, J17 CAN Output, J18 Conn_01x06, J19 Conn_02x05_Odd_Even, J2 CAN Input, J20 Conn_02x05_Odd_Even, J21 Conn_01x06, J3 Encoder 1, J4 Encoder 2, J5 Conn_01x06, J6 CPU2 USB, J7 Conn_02x05_Odd_Even, J8 Estop Conn, J9 ADC AUX 1, Q1 AO7400-VB, Q11 AO7400-VB, Q2 AO7400-VB, Q3 NCE40P05Y, Q4 LBSS139WT1G, Q7 Q_NMOS_GSD, Q8 Q_NMOS_GSD, SW1 KT11B2SAM34LFS, SW3 CONFIG SWITCH, SW4 SW_DIP_x01, SW5 KT11B2SAM34LFS, U10 TXS0101DCKR, U11 TLV1117LV33DCYR, U12 W25Q128JVSIQ, U13 W25Q128JVSIQ, U15 RP2040, U17 CA-IS3052G, U18 MCP2515-xSO, U19 RP2040, U22 ADS7822U, U23 SN74LVC1G07QDCKTQ1, U24 MT2492, U25 SN74LVC1G07QDCKTQ1, U26 ADC081S021CISD/NOPB, U27 USBLC6-2P6, U28 USBLC6-2P6, U29 USBLC6-4SC6, U3 USBLC6-4SC6, U30 USBLC6-4SC6, U31 USBLC6-4SC6, U32 TLV1117LV33DCYR, U33 TX4139, U34 LTV-208, U35 PCA9557PWR, U4 TXS0101DCKR, U43 USBLC6-4SC6, U6 SN74LVC1G07QDCKTQ1, U9 ADC081S021CISD/NOPB, Y1 12MHz, Y2 12MHz, Y3 16MHz

Commit message: Remove 2nd Motor Stuff.
Parts:
- removed C1, C8: 4.7uF 35V, Capacitor_SMD:C_0603_1608Metric, symbol Device:C
- removed C10, C11, C5, C6, C7, C9: ~, Capacitor_SMD:C_0805_2012Metric, symbol Device:C
- removed C119, C4, C43, C44, C45, C46, C47, C48, C49, C50, C51, C52, C55, C56, C67: 100n, Capacitor_SMD:C_0603_1608Metric, symbol Device:C
- removed C123, C124, C18, C20, C53, C54: 1u, Capacitor_SMD:C_0603_1608Metric, symbol Device:C
- removed C13, C86: 10u, Capacitor_SMD:C_0805_2012Metric, symbol Device:C
- removed C15: 2.2u, Capacitor_SMD:C_0603_1608Metric, symbol Device:C
- removed C19, C42: 20p, Capacitor_SMD:C_0603_1608Metric, symbol Device:C
- removed C23, C63, C64: 47p, Capacitor_SMD:C_0603_1608Metric, symbol Device:C
- removed C57, C58: 18p, Capacitor_SMD:C_0603_1608Metric, symbol Device:C
- removed C90, C91, C92: 22nF, Capacitor_SMD:C_0805_2012Metric, symbol Device:C
- removed D1, D40: ESDCAN24-2BLY, Package_TO_SOT_SMD:SOT-23, symbol Power_Protection:NUP2105L
- removed D28, D29, D30, D32: TVS 3.3V, Diode_SMD:D_SOD-523, symbol Diode:SMF54A
- removed D3: TVS 5V, Diode_SMD:D_SMA, symbol Diode:SMF54A
- removed D33, D34, D35: WS2812B, RP2040_minimal:LED_WS2812_3528_3.5x2.8mm_P1.5mm, symbol MotorBuck:WS2812B
- removed D36, D44: BAT54S, Package_TO_SOT_SMD:SOT-23, symbol Diode:BAT54S
- removed D37: B5819W SL, Diode_SMD:D_SOD-123, symbol Diode:MBR340
- removed D38: LED_GREEN, LED_SMD:LED_0805_2012Metric, symbol Device:LED
- removed D39: LED_YELLOW, LED_SMD:LED_0805_2012Metric, symbol Device:LED
- removed D41: LED_RED, LED_SMD:LED_0603_1608Metric, symbol Device:LED
- removed D45: 10V Zener, Diode_SMD:D_SOD-123, symbol Device:D_Zener
- removed FB2: 1.6Ω ±25% 1kΩ@100MHz, Inductor_SMD:L_0603_1608Metric, symbol Device:FerriteBead
- removed J10: AUX GPIO 1, parts:CONN-TH_3P-P2.54_HCTL_HC-2510-3AW, symbol Connector_Generic:Conn_01x03
- removed J11: CAN2 PLUG, parts:PINREX-744-81-04TW00 _1x04_P2.54mm_Vertical, symbol Connector_Generic:Conn_01x04
- removed J12: Conn_01x06, parts:Ckmtw-W-2510S06P_1x06_P2.54mm_Vertical, symbol Connector_Generic:Conn_01x06
- removed J13: ADC AUX 2, parts:CONN-TH_3P-P2.54_HCTL_HC-2510-3AW, symbol Connector_Generic:Conn_01x03
- removed J14: AUX GPIO 2, parts:CONN-TH_3P-P2.54_HCTL_HC-2510-3AW, symbol Connector_Generic:Conn_01x03
- removed J15: AUX Encoder, parts:CONN-TH_5P-P2.54_HCTL_HC-2510-5AW, symbol Connector_Generic:Conn_01x05
- removed J17: CAN Output, parts:M12A-08PFFR, symbol motor_parts:M12_X8_CONNECTOR
- removed J2: CAN Input, parts:M12A-08PFFR, symbol motor_parts:M12_X8_CONNECTOR
- removed J4: Encoder 2, parts:Ckmtw-W-2510S06P_1x06_P2.54mm_Vertical, symbol Connector_Generic:Conn_01x06
- removed J6: CPU2 USB, Connector_USB:USB_C_Receptacle_XKB_U262-16XN-4BVC11, symbol Connector:USB_C_Receptacle_USB2.0
- removed J8: Estop Conn, parts:BOOMELE-2510-3A_1x03_P2.54mm_Vertical, symbol Connector_Generic:Conn_01x03
- removed J9: ADC AUX 1, parts:CONN-TH_3P-P2.54_HCTL_HC-2510-3AW, symbol Connector_Generic:Conn_01x03
- removed JP1, JP14, JP15, JP4, JP5, JP6, JP7: SolderJumper_2_Open, Jumper:SolderJumper-2_P1.3mm_Open_RoundedPad1.0x1.5mm, symbol Jumper:SolderJumper_2_Open
- removed JP10, JP11, JP12, JP13, JP3: SolderJumper_3_Open, Jumper:SolderJumper-3_P1.3mm_Open_RoundedPad1.0x1.5mm, symbol Jumper:SolderJumper_3_Open
- removed Q1, Q11, Q2: AO7400-VB, Package_TO_SOT_SMD:SOT-323_SC-70, symbol Transistor_FET:AO3400A
- removed Q7, Q8: Q_NMOS_GSD, Package_TO_SOT_SMD:SOT-23, symbol Device:Q_NMOS_GSD
- removed R1, R3, R4, R5, R6, R7: ~, Resistor_SMD:R_0805_2012Metric, symbol MotorController:TAYLOR_RESISTOR
- removed R10: 510R, Resistor_SMD:R_0603_1608Metric, symbol MotorController:TAYLOR_RESISTOR
- removed R100, R48, R75, R9: 120R, Resistor_SMD:R_0603_1608Metric, symbol MotorController:TAYLOR_RESISTOR
- removed R103: 100k, Resistor_SMD:R_0603_1608Metric, symbol MotorController:TAYLOR_RESISTOR
- removed R11, R12, R13, R137, R138, R14, R17, R18, R19, R53, R55, R57, R72, R74, R79, R8: 10k, Resistor_SMD:R_0603_1608Metric, symbol MotorController:TAYLOR_RESISTOR
- removed R23: 50k 0.1%, Resistor_SMD:R_0603_1608Metric, symbol MotorController:TAYLOR_RESISTOR
- removed R40, R46, R49, R76: 5.1k, Resistor_SMD:R_0603_1608Metric, symbol Device:R
- removed R47, R66: 1.1k, Resistor_SMD:R_0603_1608Metric, symbol Device:R
- removed R51: DNS, Resistor_SMD:R_0402_1005Metric, symbol Device:R
- removed R67, R70, R71: 27R, Resistor_SMD:R_0603_1608Metric, symbol Device:R
- removed R68: 56R, Resistor_SMD:R_0603_1608Metric, symbol Device:R
- removed R77: 82R, Resistor_SMD:R_0603_1608Metric, symbol MotorController:TAYLOR_RESISTOR
- removed R99: 10.2R, Resistor_SMD:R_0603_1608Metric, symbol MotorController:TAYLOR_RESISTOR
- removed SW3: CONFIG SWITCH, Button_Switch_SMD:SW_DIP_SPSTx06_Slide_KingTek_DSHP06TS_W7.62mm_P1.27mm, symbol Switch:SW_DIP_x06
- removed SW4: SW_DIP_x01, parts:SW-SMD_DSHP01TSGER, symbol Switch:SW_DIP_x01
- removed SW5: KT11B2SAM34LFS, parts:KEY-SMD_KT11B2SAM34LFS, symbol motor_parts:SW_Push_2-4
- removed TP1, TP12, TP23, TP24, TP25, TP26, TP27, TP28, TP29, TP3, TP30, TP31, TP32, TP33, TP34, TP35, TP36, TP37, TP38, TP39, TP4, TP43, TP44, TP45, TP46, TP47, TP48, TP49, TP50, TP51, TP53, TP54, TP55, TP56, TP57, TP59, TP60, TP61, TP63, TP7, TP8, TP9: TestPoint, TestPoint:TestPoint_Pad_D1.0mm, symbol Connector:TestPoint
- removed TP2: TestPoint, TestPoint:TestPoint_Loop_D2.60mm_Drill1.6mm_Beaded, symbol Connector:TestPoint
- removed TP22: TestPoint, TestPoint:TestPoint_Keystone_5019_Minature, symbol Connector:TestPoint
- removed U10, U4: TXS0101DCKR, Package_TO_SOT_SMD:SOT-363_SC-70-6, symbol MotorBuck:level_shifter
- removed U13: W25Q128JVSIQ, Package_SO:SOIC-8_5.23x5.23mm_P1.27mm, symbol Memory_Flash:W25Q128JVS
- removed U16: ~, Package_SO:SOP-4_4.4x2.6mm_P1.27mm, symbol Isolator:SFH617A-1X007T
- removed U17: CA-IS3052G, Package_SO:SOIC-8_7.5x5.85mm_P1.27mm, symbol motor_parts:CA-IS3052G
- removed U18: MCP2515-xSO, Package_SO:SOIC-18W_7.5x11.6mm_P1.27mm, symbol Interface_CAN_LIN:MCP2515-xSO
- removed U19: RP2040, RP2040_minimal:RP2040-QFN-56, symbol MCU_RaspberryPi_RP2040:RP2040
- removed U2: ~, driver_module:driver_module, symbol driver_module:Driver
- removed U23, U25, U6: SN74LVC1G07QDCKTQ1, Package_TO_SOT_SMD:SOT-353_SC-70-5, symbol acorn-motherboard:SN74LVC1G07QDCKTQ1
- removed U26, U9: ADC081S021CISD/NOPB, Package_TO_SOT_SMD:SOT-23-6, symbol 2022-06-16_01-48-54:ADC081S021CISD/NOPB
- removed U28: USBLC6-2P6, Package_TO_SOT_SMD:SOT-666, symbol Power_Protection:USBLC6-2P6
- removed U3, U30, U31: USBLC6-4SC6, Package_TO_SOT_SMD:SOT-23-6, symbol Power_Protection:USBLC6-4SC6
- removed U34: LTV-208, parts:SSOP-8_3.91x5.84x3.18mm_P1.27mm, symbol Isolator:LTV-827S
- removed U35: PCA9557PWR, Package_SO:TSSOP-16_4.4x5mm_P0.65mm, symbol Interface_Expansion:PCA9557PW
- removed Y2: 12MHz, Crystal:Crystal_SMD_3225-4Pin_3.2x2.5mm, symbol Device:Crystal_GND24
- removed Y3: 16MHz, Crystal:Crystal_SMD_3225-4Pin_3.2x2.5mm, symbol Device:Crystal_GND24
Connections:
- net ENC2_CS: no longer names the net of U15.28 (GPIO17)
- net ENC2_RX: no longer names the net of U15.27 (GPIO16)
- net ENC2_SCK: no longer names the net of U15.29 (GPIO18)
- net ESTOP: no longer names the net of U15.30 (GPIO19)
- net M2A_PWM_H: no longer names the net of U15.17 (GPIO14)
- net M2A_PWM_L\: no longer names the net of U15.18 (GPIO15)
- net M2A_SENSE: no longer names the net of U15.38 (GPIO26_ADC0)
- net M2B_PWM_H: no longer names the net of U15.15 (GPIO12)
- net M2B_PWM_L\: no longer names the net of U15.16 (GPIO13)
- net M2C_PWM_H: no longer names the net of U15.13 (GPIO10)
- net M2C_PWM_L\: no longer names the net of U15.14 (GPIO11)
- net M2C_SENSE: no longer names the net of U15.39 (GPIO27_ADC1)
- no-connect marks 5 -> 0
Other:
- note removed: "100ms RC timer for board rev identification"
- note removed: "CAN Bus"
- note removed: "CAN bus ID"
- note removed: "CAN-ID"
- note removed: "CPU2 - Communications and GPIO"
- note removed: "CPU2 and EXT IO"
- note removed: "Can optionally drive a 5V LED strip."
- note removed: "Configuration"
- note removed: "Debug"
- note removed: "External GPIO"
- note removed: "External Thermistor Connections (to encoder ports)"
- note removed: "Jumpers enable additional filtering for hall sensors."
- note removed: "LEDs"
- note removed: "Make sure C54 is close to pin 44 of RP2040"
- note removed: "Onboard Thermistors"
- note removed: "Optional 12V fan control or normal extra GPIO"
- note removed: "Optional remote enable"
- note removed: "PWR LED"
- note removed: "When selected via SW4, the motherboard must send 5v over the CAN bus circuit to enable the power supply."
- note removed: "and extra on-board IO for future use."
- note removed: "isolation bypass"
