File: RP2040_base/RP2040_base.kicad_pcb (KiCad board)
At the start: 4 copper layers, 94.4 x 72.8 mm, 325 parts, among them J1 CPU1 USB, J10 AUX GPIO 1, J11 CAN2 PLUG, J12 Conn_01x06, J13 ADC AUX 2, J14 AUX GPIO 2, J15 AUX Encoder, J16 Conn_02x05_Odd_Even, J17 CAN Output, J18 Conn_01x06, J19 Conn_02x05_Odd_Even, J2 CAN Input, J20 Conn_02x05_Odd_Even, J21 Conn_01x06, J3 Encoder 1, J4 Encoder 2, J5 Conn_01x06, J6 CPU2 USB, J7 Conn_02x05_Odd_Even, J8 Estop Conn, J9 ADC AUX 1, Q1 AO7400-VB, Q11 AO7400-VB, Q2 AO7400-VB, Q3 AO7401, Q4 LBSS139WT1G, Q7 Q_NMOS_GSD, Q8 Q_NMOS_GSD, SW1 KT11B2SAM34LFS, SW3 CONFIG SWITCH, SW4 SW_DIP_x01, SW5 KT11B2SAM34LFS, U10 TXS0101DCKR, U11 TLV1117LV33DCYR, U12 W25Q128JVSIQ, U13 W25Q128JVSIQ, U15 RP2040, U17 CA-IS3052G, U18 MCP2515-xSO, U19 RP2040, U22 ADS7822U, U23 SN74LVC1G07QDCKTQ1, U24 MT2492, U25 SN74LVC1G07QDCKTQ1, U26 ADC081S021CISD/NOPB, U27 USBLC6-2P6, U28 USBLC6-2P6, U29 USBLC6-4SC6, U3 USBLC6-4SC6, U30 USBLC6-4SC6, U31 USBLC6-4SC6, U32 TLV1117LV33DCYR, U33 TX4139, U34 LTV-208, U35 PCA9557PWR, U4 TXS0101DCKR, U43 USBLC6-4SC6, U6 SN74LVC1G07QDCKTQ1, U9 ADC081S021CISD/NOPB, Y1 12MHz, Y2 12MHz, Y3 16MHz

Commit message: Make V1 Motor Board.
Parts:
- removed the G*** at (163.2, 74.8)
- removed the G*** at (142.8, 72.8)
- removed the G*** at (154.2, 70.8)
- removed J16, J19, J20, J7: Conn_02x05_Odd_Even, Connector_PinSocket_2.54mm:PinSocket_2x05_P2.54mm_Vertical
- removed J18, J21: Conn_01x06, Connector_PinSocket_2.54mm:PinSocket_1x06_P2.54mm_Vertical
Other:
- board text removed: "Designed by Sequoia Hope Alexander For Twisted Fields"
- board text removed: "Love everyone."
- board text removed: "Many thanks to Daniel Theobald and our supporters on"
- board text removed: "Please clone this board!"
- board text removed: "Thanks Katie for all your help!"
- board text removed: "The smallest change can be the beginning of something big."
- board text removed: "We are all star stuff."
- board text removed: "We need your help. Fork the design and make it yours."
- board text removed: "You can do it!"
- board text removed: "open collective for funding this work!"
